File: bottom-plate/switch42.kicad_pcb (KiCad board)
At the start: 2 copper layers, 128.6 x 66.7 mm, 4 parts

Commit message: Update footprints
Parts:
- Ref** (x4): moved to B.Cu
Changed lines of the file:
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@@
     (uvia_drill 0.1)
   )
-  (module phi-kbd-library:M2_SCREW_HOLE (layer F.Cu)
+  (module phi-kbd-library:M2_SCREW_HOLE (layer B.Cu)
     (at 74.922376 64.827818)
     (descr "Mounting Hole 2.2mm, no annular, M2")
     (tags "mounting hole 2.2mm no annular m2")
     (attr virtual)
-    (fp_text reference Ref** (at 0 -3.2) (layer F.Fab)
-      (effects (font (size 1 1) (thickness 0.15)))
+    (fp_text reference Ref** (at 0 3.2) (layer B.Fab)
+      (effects (font (size 1 1) (thickness 0.15)) (justify mirror))
     )
-    (fp_text value Val** (at 0 3.2) (layer F.Fab)
-      (effects (font (size 1 1) (thickness 0.15)))
+    (fp_text value Val** (at 0 -3.2) (layer B.Fab)
+      (effects (font (size 1 1) (thickness 0.15)) (justify mirror))
     )
-    (fp_text user %R (at 0.3 0) (layer F.Fab)
-      (effects (font (size 1 1) (thickness 0.15)))
+    (fp_text user %R (at 0.3 0) (layer B.Fab)
+      (effects (font (size 1 1) (thickness 0.15)) (justify mirror))
     )
     (pad "" np_thru_hole circle (at 0 0) (size 2.4 2.4) (drill 2.2) (layers *.Cu *.Mask))
+    (model ${KISYS3DMOD}/phi-kbd.3dshapes/M2_Screw.step
+      (at (xyz 0 0 0))
+      (scale (xyz 1 1 1))
+      (rotate (xyz 0 0 0))
+    )
   )
-  (module phi-kbd-library:M2_SCREW_HOLE (layer F.Cu)
+  (module phi-kbd-library:M2_SCREW_HOLE (layer B.Cu)
     (at 74.922376 90.426406)
     (descr "Mounting Hole 2.2mm, no annular, M2")
     (tags "mounting hole 2.2mm no annular m2")
     (attr virtual)
-    (fp_text reference Ref** (at 0 -3.2) (layer F.Fab)
-      (effects (font (size 1 1) (thickness 0.15)))
+    (fp_text reference Ref** (at 0 3.2) (layer B.Fab)
+      (effects (font (size 1 1) (thickness 0.15)) (justify mirror))
     )
-    (fp_text value Val** (at 0 3.2) (layer F.Fab)
-      (effects (font (size 1 1) (thickness 0.15)))
+    (fp_text value Val** (at 0 -3.2) (layer B.Fab)
+      (effects (font (size 1 1) (thickness 0.15)) (justify mirror))
     )
-    (fp_text user %R (at 0.3 0) (layer F.Fab)
-      (effects (font (size 1 1) (thickness 0.15)))
+    (fp_text user %R (at 0.3 0) (layer B.Fab)
+      (effects (font (size 1 1) (thickness 0.15)) (justify mirror))
     )
     (pad "" np_thru_hole circle (at 0 0) (size 2.4 2.4) (drill 2.2) (layers *.Cu *.Mask))
+    (model ${KISYS3DMOD}/phi-kbd.3dshapes/M2_Screw.step
+      (at (xyz 0 0 0))
+      (scale (xyz 1 1 1))
+      (rotate (xyz 0 0 0))
+    )
   )
-  (module phi-kbd-library:M2_SCREW_HOLE (layer F.Cu)
+  (module phi-kbd-library:M2_SCREW_HOLE (layer B.Cu)
     (at 193.39026 68.697372)
     (descr "Mounting Hole 2.2mm, no annular, M2")
     (tags "mounting hole 2.2mm no annular m2")
     (attr virtual)
-    (fp_text reference Ref** (at 0 -3.2) (layer F.Fab)
-      (effects (font (size 1 1) (thickness 0.15)))
+    (fp_text reference Ref** (at 0 3.2) (layer B.Fab)
+      (effects (font (size 1 1) (thickness 0.15)) (justify mirror))
     )
-    (fp_text value Val** (at 0 3.2) (layer F.Fab)
-      (effects (font (size 1 1) (thickness 0.15)))
+    (fp_text value Val** (at 0 -3.2) (layer B.Fab)
+      (effects (font (size 1 1) (thickness 0.15)) (justify mirror))
     )
-    (fp_text user %R (at 0.3 0) (layer F.Fab)
-      (effects (font (size 1 1) (thickness 0.15)))
+    (fp_text user %R (at 0.3 0) (layer B.Fab)
+      (effects (font (size 1 1) (thickness 0.15)) (justify mirror))
     )
     (pad "" np_thru_hole circle (at 0 0) (size 2.4 2.4) (drill 2.2) (layers *.Cu *.Mask))
+    (model ${KISYS3DMOD}/phi-kbd.3dshapes/M2_Screw.step
+      (at (xyz 0 0 0))
+      (scale (xyz 1 1 1))
+      (rotate (xyz 0 0 0))
+    )
   )
-  (module phi-kbd-library:M2_SCREW_HOLE (layer F.Cu)
+  (module phi-kbd-library:M2_SCREW_HOLE (layer B.Cu)
     (at 193.39026 96.081908)
     (descr "Mounting Hole 2.2mm, no annular, M2")
     (tags "mounting hole 2.2mm no annular m2")
     (attr virtual)
-    (fp_text reference Ref** (at 0 -3.2) (layer F.Fab)
-      (effects (font (size 1 1) (thickness 0.15)))
+    (fp_text reference Ref** (at 0 3.2) (layer B.Fab)
+      (effects (font (size 1 1) (thickness 0.15)) (justify mirror))
     )
-    (fp_text value Val** (at 0 3.2) (layer F.Fab)
-      (effects (font (size 1 1) (thickness 0.15)))
+    (fp_text value Val** (at 0 -3.2) (layer B.Fab)
+      (effects (font (size 1 1) (thickness 0.15)) (justify mirror))
     )
-    (fp_text user %R (at 0.3 0) (layer F.Fab)
-      (effects (font (size 1 1) (thickness 0.15)))
+    (fp_text user %R (at 0.3 0) (layer B.Fab)
+      (effects (font (size 1 1) (thickness 0.15)) (justify mirror))
     )
     (pad "" np_thru_hole circle (at 0 0) (size 2.4 2.4) (drill 2.2) (layers *.Cu *.Mask))
+    (model ${KISYS3DMOD}/phi-kbd.3dshapes/M2_Screw.step
+      (at (xyz 0 0 0))
+      (scale (xyz 1 1 1))
+      (rotate (xyz 0 0 0))
+    )
   )
   (gr_line (start 78.494272 49.051944) (end 197.557472 49.051944) (layer Edge.Cuts) (width 0.1))
