File: pcb/switch42.kicad_pcb (KiCad board)
At the start: 2 copper layers, 128.6 x 66.7 mm, 43 parts, among them J1 MJ-4PP-9, SW1 SW_PUSH, SW10 SW_PUSH, SW11 SW_PUSH, SW12 SW_PUSH, SW13 SW_PUSH, SW14 SW_PUSH, SW15 SW_PUSH, SW16 SW_PUSH, SW17 SW_PUSH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

Commit message: Redraw schema and update pcb layout
Parts:
- removed Ref** (x4): Val**, phi-kbd-library:M2_SPACER_HOLE
- added D19: D, phi-kbd-library:D_TH-reversible, F.Cu at (156.0, 52.9)
- added J2: MJ-4PP-9, phi-kbd-library:MJ-4PP-9-irreversible, B.Cu at (178.0, 52.6)
- added SW20: SW_PUSH, phi-kbd-library:MX_1.00u-irreversible, B.Cu at (165.5, 44.6)
- added SW21: SW_PUSH, phi-kbd-library:MX_1.25u-irreversible, B.Cu at (63.1, 63.6)
- added SW22: SW_PUSH, phi-kbd-library:MX_1.50u-irreversible, B.Cu at (65.5, 82.7)
- added SW23: SW_PUSH, phi-kbd-library:MX_1.50u-irreversible, B.Cu at (65.5, 44.6)
- added SW24: SW_PUSH, phi-kbd-library:MX_1.00u-irreversible, B.Cu at (84.6, 63.6)
- added SW25: SW_PUSH, phi-kbd-library:MX_1.00u-irreversible, B.Cu at (89.3, 82.7)
- added SW26: SW_PUSH, phi-kbd-library:MX_1.00u-irreversible, B.Cu at (89.3, 44.6)
- added SW27: SW_PUSH, phi-kbd-library:MX_1.00u-irreversible, B.Cu at (103.6, 63.6)
- added SW28: SW_PUSH, phi-kbd-library:MX_1.00u-irreversible, B.Cu at (108.4, 82.7)
- added SW29: SW_PUSH, phi-kbd-library:MX_1.00u-irreversible, B.Cu at (108.4, 44.6)
- added SW30: SW_PUSH, phi-kbd-library:MX_1.00u-irreversible, B.Cu at (122.7, 63.6)
- added SW31: SW_PUSH, phi-kbd-library:MX_1.00u-irreversible, B.Cu at (127.4, 82.7)
- added SW32: SW_PUSH, phi-kbd-library:MX_1.00u-irreversible, B.Cu at (127.4, 44.6)
- added SW33: SW_PUSH, phi-kbd-library:MX_1.00u-irreversible, B.Cu at (141.7, 63.6)
- added SW34: SW_PUSH, phi-kbd-library:MX_1.00u-irreversible, B.Cu at (146.5, 82.7)
- added SW35: SW_PUSH, phi-kbd-library:MX_1.00u-irreversible, B.Cu at (146.5, 44.6)
- added SW36: SW_PUSH, phi-kbd-library:MX_1.00u-irreversible, B.Cu at (160.8, 63.6)
- added SW37: SW_PUSH, phi-kbd-library:MX_1.00u-irreversible, B.Cu at (165.5, 82.7)
- J1: footprint phi-kbd-library:MJ-4PP-9-reversible -> phi-kbd-library:MJ-4PP-9-irreversible; moved to F.Cu
- SW10, SW11, SW12, SW13, SW14, SW15, SW16, SW17, SW18, SW5, SW6, SW7, SW8, SW9: footprint phi-kbd-library:MX_1.00u-reversible -> phi-kbd-library:MX_1.00u-irreversible
- SW19, SW2: footprint phi-kbd-library:MX_1.25u-reversible -> phi-kbd-library:MX_1.00u-irreversible
- SW3: footprint phi-kbd-library:MX_1.00u-reversible -> phi-kbd-library:MX_1.25u-irreversible
- SW4: footprint phi-kbd-library:MX_1.00u-reversible -> phi-kbd-library:MX_1.50u-irreversible
- moved J1 37.4 mm to (178.0, 54.1)
- moved D16 37.2 mm to (141.7, 52.9), turned to 180 degrees
- moved SW14 35.0 mm to (137.0, 44.6)
- moved SW17 35.0 mm to (156.0, 44.6)
- moved SW5 35.0 mm to (79.8, 44.6)
- moved SW8 35.0 mm to (98.9, 44.6)
- moved SW11 35.0 mm to (117.9, 44.6)
- moved D17 33.6 mm to (152.7, 63.6), turned to 90 degrees
- moved SW2 32.8 mm to (60.8, 44.6)
- moved D10 32.5 mm to (108.4, 52.9), turned to 180 degrees
- moved D13 32.5 mm to (127.4, 52.9), turned to 180 degrees
- moved D7 32.5 mm to (89.3, 52.9), turned to 180 degrees
- moved SW19 31.0 mm to (165.5, 82.7)
- moved D18 30.6 mm to (156.0, 82.7), turned to 90 degrees
- moved D4 30.2 mm to (72.7, 52.9), turned to 180 degrees
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Connections:
- net row3 renamed Net-(U1-Pad10)
- U1 pad 14: Net-(U1-Pad14) -> col6
Routing:
- net col5: track 155.9 -> 0.00 mm
- net row0: track 146.1 -> 0.00 mm
- net GND: track 143.0 -> 0.00 mm
- net col4: track 138.4 -> 0.00 mm
- net VCC: track 133.1 -> 0.00 mm
- net row2: track 126.7 -> 0.00 mm
- net reset: track 124.7 -> 0.00 mm
- net data: track 124.6 -> 0.00 mm
- net col3: track 121.9 -> 0.00 mm
- net row1: track 108.8 -> 0.00 mm
- net col2: track 95.9 -> 0.00 mm
- net col1: track 88.3 -> 0.00 mm
- net col0: track 54.2 -> 0.00 mm
- net Net-(D2-Pad2): track 29.0 -> 0.00 mm
- net Net-(D18-Pad2): track 20.9 -> 0.00 mm
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- removed copper zone on B.Cu, net GND
- removed copper zone on F.Cu, net GND
Other:
- board size 128.6 x 66.7 mm -> 130.7 x 57.2 mm
- board text removed: "KASTOR Keyboard rev.1 by zk-phi"

Commit message: Complate wiring
Parts:
- D1, D10, D11, D12, D13, D14, D15, D16, D17, D18, D19, D2, D3, D4, D5, D6, D7, D8, D9: footprint phi-kbd-library:D_TH-reversible -> phi-kbd-library:D_SMD-reversible
- moved D6 14.3 mm to (93.2, 86.8)
- moved D12 14.0 mm to (131.3, 86.8)
- moved D15 14.0 mm to (150.4, 86.8)
- moved D18 14.0 mm to (169.4, 86.8)
- moved D9 14.0 mm to (112.3, 86.8)
- moved D17 12.6 mm to (164.6, 67.8)
- moved D2 12.6 mm to (80.7, 67.8)
- moved D4 11.2 mm to (83.1, 48.7), turned to 90 degrees
- moved D5 8.27 mm to (88.4, 67.8)
- moved D3 7.27 mm to (69.4, 86.8)
- moved D8 7.02 mm to (107.5, 67.8)
- moved D11 7.02 mm to (126.5, 67.8)
- moved D10 6.33 mm to (103.6, 48.7), turned to 90 degrees
- moved D13 6.33 mm to (122.7, 48.7), turned to 90 degrees
- moved D19 6.33 mm to (160.8, 48.7), turned to 90 degrees
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Routing:
- net row2: track 0.00 -> 238.4 mm
- net data: track 0.00 -> 145.1 mm
- net col5: track 0.00 -> 140.4 mm, vias 0 -> 1
- net row0: track 0.00 -> 129.5 mm, vias 0 -> 6
- net col4: track 0.00 -> 123.9 mm, vias 0 -> 1
- net VCC: track 0.00 -> 120.0 mm
- net reset: track 0.00 -> 117.7 mm
- net row1: track 0.00 -> 114.8 mm, vias 0 -> 5
- net col3: track 0.00 -> 107.4 mm, vias 0 -> 1
- net col6: track 0.00 -> 100.4 mm, vias 0 -> 1
- net col2: track 0.00 -> 90.9 mm, vias 0 -> 1
- net col0: track 0.00 -> 72.5 mm
- net col1: track 0.00 -> 71.4 mm, vias 0 -> 1
- net Net-(D2-Pad2): track 0.00 -> 41.3 mm
- net Net-(D1-Pad2): track 0.00 -> 38.3 mm
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- added copper zone on B.Cu, net GND
- added copper zone on F.Cu, net GND

Commit message: Add keyboard name silk to the pcb
Other:
- board text added: "K A S T O R k e y b o a r d P C B - r e v . 2"
Changed lines of the file:
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@@
   (general
     (thickness 1.6)
-    (drawings 26)
+    (drawings 28)
     (tracks 387)
     (zones 0)
@@
     )
   )
+  (gr_text "K A S T O R   k e y b o a r d    P C B - r e v . 2" (at 113.144608 73.152168) (layer B.SilkS)
+    (effects (font (size 1.5 1.5) (thickness 0.3)) (justify mirror))
+  )
+  (gr_text "K A S T O R   k e y b o a r d    P C B - r e v . 2" (at 113.144608 73.152168) (layer F.SilkS)
+    (effects (font (size 1.5 1.5) (thickness 0.3)))
+  )
   (gr_line (start 46.171558 68.091982) (end 46.171558 97.262466) (layer F.Fab) (width 0.12))
